File: rgb-segment.sch (EAGLE design)
At the start: 33 parts

Commit message: Completition of the schema - First version of the board - 17-07-2016
Parts:
- removed LED29: WS2812B_5050N, adafruit:WS2812B_5050N
- added C10, C11, C12, C13, C14, C15, C16, C17, C18, C19, C20, C21, C22, C23, C24, C25, C26, C27, C28, C6, C7, C8, C9: 0.1uF, rcl:C-EUC0805
- added C29: (no value), SparkFun-Passives:CAP_POLG
- added D1: (no value), diode:DIODE-DO214AC
- added DIJ: Diode-Control, SparkFun-Passives:JUMPER-PAD-3-2OF3_NC_BY_TRACE_SMALL
- added LED1: WS2812B_5050N, adafruit:WS2812B_5050N
- added PIN_IN, PIN_OUT: (no value), pinhead:PINHD-1X3
Connections:
- removed net N$3 (its old number): LED3.DI, LED4.DO
- removed net N$41 (its old number): LED13.DI, LED14.DO
- removed net N$5 (its old number): LED2.DI, LED3.DO
- removed net N$55 (its old number): LED17.DI, LED2.DO
- removed net N$59 (its old number): LED16.DI, LED17.DO
- removed net N$62 (its old number): LED15.DI, LED16.DO
- removed net N$65 (its old number): LED14.DI, LED15.DO
- removed net N$70 (its old number): LED12.DI, LED13.DO
- removed net N$72 (its old number): LED11.DI, LED12.DO
- removed net N$74 (its old number): LED10.DI, LED11.DO
- new net +5V: C10.2, C11.2, C12.2, C13.2, C14.2, C15.2, C16.2, C17.2, C18.2, C19.2, C2.1, C20.2, C21.1, C22.1, C23.1, C24.1, C25.1, C26.1, C27.1, C28.1, C29.+, C3.1, C4.1, C5.2, C6.2, C7.2, C8.2, C9.2, D1.A, DIJ.3, LED10.VDD, LED11.VDD, LED12.VDD, LED13.VDD, LED14.VDD, LED15.VDD, LED16.VDD, LED17.VDD, LED18.VDD, LED19.VDD, LED2.VDD, LED20.VDD, LED21.VDD, LED22.VDD, LED23.VDD, LED24.VDD, LED25.VDD, LED26.VDD, LED27.VDD, LED28.VDD, LED3.VDD, LED5.VDD, LED6.VDD, LED7.VDD, LED8.VDD, LED9.VDD, PIN_IN.3, PIN_OUT.1
- new net N$10: D1.C, DIJ.1
- new net N$12: LED5.DO, LED6.DI
- new net N$14: LED6.DO, LED7.DI
- new net N$16: LED7.DO, LED8.DI
- new net N$17: LED8.DO, LED9.DI
- new net N$18: LED28.DO, PIN_OUT.2
- new net N$19: LED4.DO, LED5.DI
- new net N$2: LED4.VDD
- new net N$21: LED3.DO, LED4.DI
- new net N$23: LED10.DI, LED9.DO
- new net N$24: LED10.DO, LED11.DI
- new net N$26: LED2.DO, LED3.DI
- new net N$28: LED1.DO, LED2.DI
- new net N$4: LED1.DI, PIN_IN.2
- new net N$61: C14.1
- new net N$9: C1.1, DIJ.2, LED1.VDD
- net AGND: now also C1.2, C10.1, C11.1, C12.1, C13.1, C15.1, C16.1, C17.1, C18.1, C19.1, C2.2, C20.1, C21.2, C22.2, C23.2, C24.2, C25.2, C26.2, C27.2, C28.2, C29.-, C3.2, C4.2, C5.1, C6.1, C7.1, C8.1, C9.1, LED1.GND, PIN_IN.1, PIN_OUT.3; no longer LED29.GND
- net N$1: now also LED17.DO, LED18.DI; no longer LED4.DI, LED5.DO
- net N$30: now also LED11.DO, LED12.DI; no longer LED28.DO, LED29.DI
- net N$33: now also LED12.DO, LED13.DI; no longer LED29.DO, LED9.DI
- net N$42: now also LED13.DO, LED14.DI; no longer LED8.DI, LED9.DO
- net N$44: now also LED14.DO, LED15.DI; no longer LED7.DI, LED8.DO
- net N$46: now also LED15.DO, LED16.DI; no longer LED6.DI, LED7.DO
- net N$48: now also LED16.DO, LED17.DI; no longer LED5.DI, LED6.DO
Other:
- moved on the sheet: C5
